File: inkBT.kicad_sch (KiCad schematic)
At the start: 4 parts, among them J1 AudioJack2_Ground, U1 LM2596S-3.3, U2 ESP32-WROOM-32, U3 PCM5102A

Commit message: a
Connections:
- net GND: no longer U2.1 (GND), U2.15 (GND), U2.38 (GND), U2.39 (GND), U3.19 (DGND)
- new net: U2.1 (GND), U2.15 (GND), U2.38 (GND), U2.39 (GND)
- now unconnected: U1.2 (OUT), U2.2 (VDD), U3.20 (DVDD), U3.8 (AVDD)
Other:
- moved on the sheet: U1
Changed lines of the file:
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@@
 	(generator_version "10.0")
 	(paper "A4")
-	(junction
-		(at 245.11 142.24)
-		(diameter 0)
-		(color 0 0 0 0)
-	)
-	(junction
-		(at 248.92 83.82)
-		(diameter 0)
-		(color 0 0 0 0)
-	)
-	(junction
-		(at 228.6 160.02)
-		(diameter 0)
-		(color 0 0 0 0)
-	)
-	(wire
-		(pts
-			(xy 196.85 71.12) (xy 196.85 60.96)
-		)
-		(stroke
-			(width 0)
-			(type default)
-		)
-	)
-	(wire
-		(pts
-			(xy 196.85 60.96) (xy 248.92 60.96)
-		)
-		(stroke
-			(width 0)
-			(type default)
-		)
-	)
-	(wire
-		(pts
-			(xy 248.92 83.82) (xy 248.92 91.44)
-		)
-		(stroke
-			(width 0)
-			(type default)
-		)
-	)
 	(wire
 		(pts
@@
 	(wire
 		(pts
-			(xy 271.78 154.94) (xy 271.78 83.82)
-		)
-		(stroke
-			(width 0)
-			(type default)
-		)
-	)
-	(wire
-		(pts
-			(xy 245.11 124.46) (xy 245.11 142.24)
-		)
-		(stroke
-			(width 0)
-			(type default)
-		)
-	)
-	(wire
-		(pts
-			(xy 217.17 161.29) (xy 210.82 161.29)
-		)
-		(stroke
-			(width 0)
-			(type default)
-		)
-	)
-	(wire
-		(pts
-			(xy 245.11 160.02) (xy 228.6 160.02)
-		)
-		(stroke
-			(width 0)
-			(type default)
-		)
-	)
-	(wire
-		(pts
 			(xy 247.65 127) (xy 247.65 124.46)
 		)
@@
 	(wire
 		(pts
-			(xy 248.92 91.44) (xy 247.65 91.44)
-		)
-		(stroke
-			(width 0)
-			(type default)
-		)
-	)
-	(wire
-		(pts
-			(xy 241.3 154.94) (xy 271.78 154.94)
-		)
-		(stroke
-			(width 0)
-			(type default)
-		)
-	)
-	(wire
-		(pts
-			(xy 210.82 149.86) (xy 215.9 149.86)
-		)
-		(stroke
-			(width 0)
-			(type default)
-		)
-	)
-	(wire
-		(pts
-			(xy 245.11 142.24) (xy 245.11 160.02)
-		)
-		(stroke
-			(width 0)
-			(type default)
-		)
-	)
-	(wire
-		(pts
-			(xy 210.82 161.29) (xy 210.82 149.86)
+			(xy 130.81 176.53) (xy 132.08 176.53)
 		)
 		(stroke
@@
 	(wire
 		(pts
-			(xy 245.11 83.82) (xy 245.11 91.44)
-		)
-		(stroke
-			(width 0)
-			(type default)
-		)
-	)
-	(wire
-		(pts
-			(xy 248.92 83.82) (xy 245.11 83.82)
+			(xy 130.81 190.5) (xy 130.81 176.53)
 		)
 		(stroke
@@
 	(wire
 		(pts
-			(xy 271.78 83.82) (xy 248.92 83.82)
-		)
-		(stroke
-			(width 0)
-			(type default)
-		)
-	)
-	(wire
-		(pts
-			(xy 248.92 60.96) (xy 248.92 83.82)
-		)
-		(stroke
-			(width 0)
-			(type default)
-		)
-	)
-	(wire
-		(pts
 			(xy 259.08 118.11) (xy 267.97 118.11)
 		)
@@
 	(wire
 		(pts
-			(xy 228.6 160.02) (xy 228.6 161.29)
+			(xy 144.78 186.69) (xy 144.78 190.5)
 		)
 		(stroke
@@
 		(pts
 			(xy 260.35 99.06) (xy 257.81 99.06)
-		)
-		(stroke
-			(width 0)
-			(type default)
-		)
-	)
-	(wire
-		(pts
-			(xy 196.85 142.24) (xy 245.11 142.24)
 		)
 		(stroke
@@
 	(symbol
 		(lib_id "power:+12V")
-		(at 217.17 161.29 180)
+		(at 130.81 190.5 180)
 		(unit 1)
 		(body_style 1)
@@
 		(fields_autoplaced yes)
 		(property "Reference" "#PWR02"
-			(at 217.17 157.48 0)
+			(at 130.81 186.69 0)
 			(hide yes)
 			(show_name no)
@@
 		)
 		(property "Value" "+12V"
-			(at 217.17 166.37 0)
+			(at 130.81 195.58 0)
 			(show_name no)
 			(do_not_autoplace no)
@@
 		)
 		(property "Footprint" ""
-			(at 217.17 161.29 0)
+			(at 130.81 190.5 0)
 			(hide yes)
 			(show_name no)
@@
 		)
 		(property "Datasheet" ""
-			(at 217.17 161.29 0)
+			(at 130.81 190.5 0)
 			(hide yes)
 			(show_name no)
@@
 		)
 		(property "Description" ""
-			(at 217.17 161.29 0)
+			(at 130.81 190.5 0)
 			(show_name no)
 			(do_not_autoplace no)
@@
 	(symbol
 		(lib_id "Regulator_Switching:LM2596S-3.3")
-		(at 228.6 152.4 0)
+		(at 144.78 179.07 0)
 		(unit 1)
 		(body_style 1)
@@
 		(fields_autoplaced yes)
 		(property "Reference" "U1"
-			(at 228.6 142.24 0)
+			(at 144.78 168.91 0)
 			(show_name no)
 			(do_not_autoplace no)
@@
 		)
 		(property "Value" "LM2596S-3.3"
-			(at 228.6 144.78 0)
+			(at 144.78 171.45 0)
 			(show_name no)
 			(do_not_autoplace no)
@@
 		)
 		(property "Footprint" "Package_TO_SOT_SMD:TO-263-5_TabPin3"
-			(at 229.87 158.75 0)
+			(at 146.05 185.42 0)
 			(hide yes)
 			(show_name no)
@@
 		)
 		(property "Datasheet" "http://www.ti.com/lit/ds/symlink/lm2596.pdf"
-			(at 228.6 152.4 0)
+			(at 144.78 179.07 0)
 			(hide yes)
 			(show_name no)
@@
 		)
 		(property "Description" ""
-			(at 228.6 152.4 0)
+			(at 144.78 179.07 0)
 			(show_name no)
 			(do_not_autoplace no)
@@
 		(property "Reference" "U3"
 			(at 249.8441 88.9 0)
+			(hide yes)
 			(show_name no)
 			(do_not_autoplace no)
@@
 	(symbol
 		(lib_id "power:GND")
-		(at 228.6 161.29 0)
+		(at 144.78 190.5 0)
 		(unit 1)
 		(body_style 1)
@@
 		(fields_autoplaced yes)
 		(property "Reference" "#PWR01"
-			(at 228.6 167.64 0)
+			(at 144.78 196.85 0)
 			(hide yes)
 			(show_name no)
@@
 		)
 		(property "Value" "GND"
-			(at 228.6 166.37 0)
+			(at 144.78 195.58 0)
 			(show_name no)
 			(do_not_autoplace no)
@@
 		)
 		(property "Footprint" ""
-			(at 228.6 161.29 0)
+			(at 144.78 190.5 0)
 			(hide yes)
 			(show_name no)
@@
 		)
 		(property "Datasheet" ""
-			(at 228.6 161.29 0)
+			(at 144.78 190.5 0)
 			(hide yes)
 			(show_name no)
@@
 		)
 		(property "Description" ""
-			(at 228.6 161.29 0)
+			(at 144.78 190.5 0)
 			(show_name no)
 			(do_not_autoplace no)
@@
 		(property "Reference" "U2"
 			(at 199.0441 68.58 0)
+			(hide yes)
 			(show_name no)
 			(do_not_autoplace no)
@@
 		(property "Value" "ESP32-WROOM-32"
 			(at 199.0441 71.12 0)
-			(show_name no)
-			(do_not_autoplace no)
+			(hide yes)
+			(show_name no)
+			(do_not_autoplace no)

Commit message: a
Parts:
- added C1, C2, C3, C4: C2.2, Package_SO:SOIC-8_3.9x4.9mm_P1.27mm, symbol Device:C
- added R1, R2: R470, symbol Device:R
Connections:
- net GND: now also J1.G, U2.1 (GND), U2.15 (GND), U2.38 (GND), U2.39 (GND), C3.2, C4.2
- net 3.3v: now reaches U1.2 (OUT)
- net 3.3v: now also U2.2 (VDD)
- net at U3.2 (CAPP): now also C1.1
- net at U3.3 (CPGND): now also C2.2
- net at U3.4 (CAPM): now also C1.2
- net at U3.5 (VNEG): now also C2.1
- net at U3.6 (OUTL): now also R2.1; no longer J1.T
- net at U3.7 (OUTR): now also R1.1; no longer J1.S
- net at U3.9 (AGND): no longer J1.G
- new net: C3.1, J1.S, R1.2
- new net: C4.1, J1.T, R2.2
Other:
- moved on the sheet: J1, U1

Commit message: a
Parts:
- added C10, C12, C5, C8: C10, Capacitor_SMD:C_1206_3216Metric_Pad1.33x1.80mm_HandSolder, symbol Device:C
- added C11, C6, C7, C9: C0.1, Capacitor_SMD:C_1206_3216Metric_Pad1.33x1.80mm_HandSolder, symbol Device:C
- added J2: Conn_01x10, symbol Connector_Generic:Conn_01x10
- added R3, R4, R5: R22, Resistor_SMD:R_1206_3216Metric_Pad1.30x1.75mm_HandSolder, symbol Device:R
- added U4: LM2596S-3.3, Package_TO_SOT_SMD:TO-263-5_TabPin3, symbol Regulator_Switching:LM2596S-3.3
- C1, C2, C3, C4: footprint Package_SO:SOIC-8_3.9x4.9mm_P1.27mm -> Capacitor_SMD:C_1206_3216Metric_Pad1.33x1.80mm_HandSolder
- J1: footprint Connector_Audio:Jack_3.5mm_QingPu_WQP-PJ398SM_Vertical_CircularHoles -> Connector_PinSocket_1.00mm:PinSocket_1x03_P1.00mm_Vertical
- R1, R2: footprint (none) -> Resistor_SMD:R_1206_3216Metric_Pad1.30x1.75mm_HandSolder
Connections:
- net +12V: now also U4.1 (VIN)
- net 3.3v: now also U3.17 (XSMT), U3.20 (DVDD), C11.2, C12.2, C7.1, C8.1
- net GND: now also U3.10 (DEMP), U3.11 (FLT), U3.12 (SCK), U3.16 (FMT), U3.19 (DGND), U3.9 (AGND), C10.2, C11.1, C12.1, C5.2, C6.2, C7.2, C8.2, C9.2, U4.3 (GND)
- net 3.3v analog: now reaches U3.1 (CPVDD)
- net 3.3v analog: now also U3.8 (AVDD), C5.1, C6.1, U4.2 (OUT)
- net at U3.13 (BCK): now also R5.2
- net at U3.14 (DIN): now also R4.2
- net at U3.15 (LRCK): now also R3.2
- net at U3.18 (LDOO): now also C10.1, C9.1
- net at U2.13 (IO14): now also J2.5 (Pin_5)
- net at U2.14 (IO12): now also J2.3 (Pin_3)
- net at U2.16 (IO13): now also J2.4 (Pin_4)
- net at U2.23 (IO15): now also J2.6 (Pin_6)
- net at U2.26 (IO4): now also J2.1 (Pin_1)
- net at U2.27 (IO16): now also J2.7 (Pin_7)
- net at U2.28 (IO17): now also J2.8 (Pin_8)
- net at U2.29 (IO5): now also J2.2 (Pin_2)
- net at U2.30 (IO18): now also J2.9 (Pin_9)
- net at U2.31 (IO19): now also J2.10 (Pin_10)
- net dac_DIN: now reaches U2.6 (IO34)
- net dac_DIN: now also R4.1
- net dac_BCK: now reaches U2.7 (IO35)
- net dac_BCK: now also R5.1
- net dac_LRCK: now reaches U2.9 (IO33)
- net dac_LRCK: now also R3.1

Commit message: a
Parts:
- removed U1, U4: LM2596S-3.3, Package_TO_SOT_SMD:TO-263-5_TabPin3, symbol Regulator_Switching:LM2596S-3.3
- added U1: LM2596S-5, Package_TO_SOT_SMD:TO-263-5_TabPin3, symbol Regulator_Switching:LM2596S-5
- added U5: LM2596S-3.3, Package_TO_SOT_SMD:TO-263-5_TabPin3, symbol Regulator_Switching:LM2596S-3.3
- added U6, U7: ME6211C33M5, Package_TO_SOT_SMD:SOT-23-5, symbol Regulator_Linear:ME6211C33M5
Connections:
- net +12V: now also U1.1 (VIN), U5.1 (VIN)
- net 3.3v: now also U5.2 (OUT); no longer C11.2, C12.2, C7.1, C8.1, U3.17 (XSMT), U3.20 (DVDD)
- net GND: now also U1.3 (GND), U5.3 (GND), U6.2 (V_{SS}), U7.2 (V_{SS})
- net EN_dac: now reaches U2.33 (IO21)
- net EN_dac: now also U6.3 (CE), U7.3 (CE)
- net 3.3v analog renamed 3.3v Adac
- net 3.3v Adac: now also U6.5 (V_{OUT})
- new net: U1.2 (OUT), U6.1 (V_{IN}), U7.1 (V_{IN})
- new net 3.3v Ddac: C11.2, C12.2, C7.1, C8.1, U3.17 (XSMT), U3.20 (DVDD), U7.5 (V_{OUT})

Commit message: a
Parts:
- added J3: Conn_01x06, Connector_PinHeader_2.00mm:PinHeader_1x06_P2.00mm_Vertical, symbol Connector_Generic:Conn_01x06
- added R6: R100, Resistor_SMD:R_1206_3216Metric_Pad1.30x1.75mm_HandSolder, symbol Device:R
- added TP1, TP2, TP3, TP4, TP5, TP6, TP7: TestPoint, TestPoint:TestPoint_Pad_D2.0mm, symbol Connector:TestPoint
- J2: footprint (none) -> Connector_PinHeader_2.00mm:PinHeader_1x10_P2.00mm_Vertical
Connections:
- net +12V: now also TP2.1
- net 3.3v: now also U2.3 (EN), TP1.1
- net 3.3v Adac: now also TP5.1
- net 3.3v Ddac: now also TP4.1
- net EN_dac: now also R6.2, TP6.1
- net GND: now also U1.5 (~{ON}/OFF), U5.5 (~{ON}/OFF), R6.1, TP3.1
- net at U1.2 (OUT), U6.1 (V_{IN}), U7.1 (V_{IN}): now also TP7.1
- net at U2.17 (SHD/SD2): now also J3.4 (Pin_4)
- net at U2.18 (SWP/SD3): now also J3.3 (Pin_3)
- net at U2.19 (SCS/CMD): now also J3.1 (Pin_1)
- net at U2.20 (SCK/CLK): now also J3.2 (Pin_2)
- net at U2.21 (SDO/SD0): now also J3.6 (Pin_6)
- net at U2.22 (SDI/SD1): now also J3.5 (Pin_5)
Other:
- moved on the sheet: C1, C10, C11, C12, C2, C3, C4, C5, C6, C7, C8, C9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

Commit message: a
Parts:
- removed J1: AudioJack2_Ground, Connector_PinSocket_1.00mm:PinSocket_1x03_P1.00mm_Vertical, symbol Connector_Audio:AudioJack2_Ground
- added J1: Conn_01x03, Connector_PinHeader_2.00mm:PinHeader_1x03_P2.00mm_Vertical, symbol Connector_Generic:Conn_01x03
Connections:
- net GND: now also J1.1 (Pin_1)
- net at C3.1, R1.2: now also J1.3 (Pin_3)
- net at C4.1, R2.2: now also J1.2 (Pin_2)
Changed lines of the file:
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@@
 	)
 	(junction
+		(at 157.48 104.14)
+		(diameter 0)
+		(color 0 0 0 0)
+	)
+	(junction
 		(at 123.19 74.93)
 		(diameter 0)
@@
 	)
 	(junction
-		(at 153.67 104.14)
-		(diameter 0)
-		(color 0 0 0 0)
-	)
-	(junction
 		(at 129.54 74.93)
 		(diameter 0)
@@
 	(wire
 		(pts
+			(xy 165.1 104.14) (xy 157.48 104.14)
+		)
+		(stroke
+			(width 0)
+			(type default)
+		)
+	)
+	(wire
+		(pts
 			(xy 121.92 81.28) (xy 119.38 81.28)
 		)
@@
 	(wire
 		(pts
+			(xy 156.21 102.87) (xy 165.1 102.87)
+		)
+		(stroke
+			(width 0)
+			(type default)
+		)
+	)
+	(wire
+		(pts
 			(xy 127 40.64) (xy 127 22.86)
 		)
@@
 	(wire
 		(pts
-			(xy 153.67 104.14) (xy 153.67 105.41)
+			(xy 165.1 104.14) (xy 165.1 105.41)
 		)
 		(stroke
@@
 	(wire
 		(pts
+			(xy 157.48 104.14) (xy 153.67 104.14)
+		)
+		(stroke
+			(width 0)
+			(type default)
+		)
+	)
+	(wire
+		(pts
 			(xy 116.84 123.19) (xy 116.84 127)
 		)
@@
 	(wire
 		(pts
-			(xy 151.13 107.95) (xy 153.67 107.95)
+			(xy 151.13 107.95) (xy 165.1 107.95)
 		)
 		(stroke
@@
 	(wire
 		(pts
-			(xy 157.48 104.14) (xy 153.67 104.14)
-		)
-		(stroke
-			(width 0)
-			(type default)
-		)
-	)
-	(wire
-		(pts
 			(xy 97.79 100.33) (xy 106.68 100.33)
 		)
@@
 		(lib_name "GND_1")
 		(lib_id "power:GND")
-		(at 158.75 100.33 180)
+		(at 156.21 102.87 180)
 		(unit 1)
 		(body_style 1)
@@
 		(fields_autoplaced yes)
 		(property "Reference" "#PWR05"
-			(at 158.75 93.98 0)
+			(at 156.21 96.52 0)
 			(hide yes)
 			(show_name no)
@@
 		)
 		(property "Value" "GND"
-			(at 158.75 95.25 0)
+			(at 156.21 97.79 0)
 			(show_name no)
 			(do_not_autoplace no)
@@
 		)
 		(property "Footprint" ""
-			(at 158.75 100.33 0)
+			(at 156.21 102.87 0)
 			(hide yes)
 			(show_name no)
@@
 		)
 		(property "Datasheet" ""
-			(at 158.75 100.33 0)
+			(at 156.21 102.87 0)
 			(hide yes)
 			(show_name no)
@@
 		)
 		(property "Description" "Power symbol creates a global label with name \"GND\" , ground"
-			(at 158.75 100.33 0)
+			(at 156.21 102.87 0)
 			(hide yes)
 			(show_name no)
@@
 	)
 	(symbol
+		(lib_id "Connector_Generic:Conn_01x03")
+		(at 170.18 105.41 0)
+		(unit 1)
+		(body_style 1)
+		(exclude_from_sim no)
+		(in_bom yes)
+		(on_board yes)
+		(in_pos_files yes)
+		(dnp no)
+		(fields_autoplaced yes)
+		(property "Reference" "J1"
+			(at 172.72 104.1399 0)
+			(show_name no)
+			(do_not_autoplace no)
+			(effects
+				(font
+					(size 1.27 1.27)
+				)
+				(justify left)
+			)
+		)
+		(property "Value" "Conn_01x03"
+			(at 172.72 106.6799 0)
+			(show_name no)
+			(do_not_autoplace no)
+			(effects
+				(font
+					(size 1.27 1.27)
+				)
+				(justify left)
+			)
+		)
+		(property "Footprint" "Connector_PinHeader_2.00mm:PinHeader_1x03_P2.00mm_Vertical"
+			(at 170.18 105.41 0)
+			(hide yes)
+			(show_name no)
+			(do_not_autoplace no)
+			(effects
+				(font
+					(size 1.27 1.27)
+				)
+			)
+		)
+		(property "Datasheet" ""
+			(at 170.18 105.41 0)
+			(hide yes)
+			(show_name no)
+			(do_not_autoplace no)
+			(effects
+				(font
+					(size 1.27 1.27)
+				)
+			)
+		)
+		(property "Description" "Generic connector, single row, 01x03, script generated (kicad-library-utils/schlib/autogen/connector/)"
+			(at 170.18 105.41 0)
+			(hide yes)
+			(show_name no)
+			(do_not_autoplace no)
+			(effects
+				(font
+					(size 1.27 1.27)
+				)
+			)
+		)
+		(pin "2"
+		)
+		(pin "1"
+		)
+		(pin "3"
+		)
+		(instances
+			(project "inkBT"
+				(path "/d639bd58-f563-44ff-a906-a8a044dd820d"
+					(reference "J1")
+					(unit 1)
+				)
+			)
+		)
+	)
+	(symbol
 		(lib_id "Device:R")
 		(at 142.24 93.98 90)
@@
 					(unit 1)
 				)
-			)
-		)
-	)
-	(symbol
-		(lib_id "Connector_Audio:AudioJack2_Ground")
-		(at 158.75 105.41 180)
-		(unit 1)
-		(body_style 1)
-		(exclude_from_sim no)
-		(in_bom yes)
-		(on_board yes)
-		(in_pos_files yes)
-		(dnp no)
-		(fields_autoplaced yes)
-		(property "Reference" "J1"
-			(at 163.83 104.775 0)
-			(show_name no)
-			(do_not_autoplace no)
-			(effects
-				(font
-					(size 1.27 1.27)
-				)
-				(justify right)
-			)
-		)
-		(property "Value" "AudioJack2_Ground"
-			(at 163.83 107.315 0)
-			(show_name no)
-			(do_not_autoplace no)
-			(effects
-				(font
-					(size 1.27 1.27)
-				)
-				(justify right)
-			)
-		)
-		(property "Footprint" "Connector_PinSocket_1.00mm:PinSocket_1x03_P1.00mm_Vertical"
-			(at 158.75 105.41 0)
-			(hide yes)
-			(show_name no)
-			(do_not_autoplace no)
-			(effects
-				(font
-					(size 1.27 1.27)
-				)
-			)
-		)
-		(property "Datasheet" ""
-			(at 158.75 105.41 0)
-			(hide yes)
-			(show_name no)
-			(do_not_autoplace no)
-			(effects
-				(font
-					(size 1.27 1.27)
-				)
-			)
-		)
-		(property "Description" ""
-			(at 158.75 105.41 0)
-			(show_name no)
-			(do_not_autoplace no)
-			(effects
-				(font
-					(size 1.27 1.27)
-				)
-			)
-		)
-		(pin "S"
-		)
-		(pin "G"
-		)
-		(pin "T"
-		)
-		(instances
-			(project "inkBT"
-				(path "/d639bd58-f563-44ff-a906-a8a044dd820d"
-					(reference "J1")
-					(unit 1)
-				)

Commit message: a
Parts:
- removed J3: Conn_01x06, Connector_PinHeader_2.00mm:PinHeader_1x06_P2.00mm_Vertical, symbol Connector_Generic:Conn_01x06
- added H1, H2, H3, H4: MountingHole_Pad, MountingHole:MountingHole_2.5mm_Pad_Via, symbol Mechanical:MountingHole_Pad
- added J3: Conn_01x02, Connector_PinHeader_2.54mm:PinHeader_1x02_P2.54mm_Vertical, symbol Connector_Generic:Conn_01x02
- added R7: R100K, Resistor_SMD:R_1206_3216Metric_Pad1.30x1.75mm_HandSolder, symbol Device:R
- renumbered C8 to C1, C9 to C10, C12 to C11, C10 to C12, C7 to C2, C6 to C3, C5 to C4, C1 to C5, C2 to C6, C3 to C7, C4 to C8, C11 to C9, J2 to J1, J1 to J2, R6 to R1, R1 to R5, R5 to R6, TP2 to TP1, TP4 to TP2, TP5 to TP3, TP1 to TP4, TP3 to TP5, TP7 to TP6, TP6 to TP7, U5 to U1, U7 to U2, U6 to U3, U1 to U4, U2 to U5, U3 to U6
Connections:
- net +12V: now also J3.1 (Pin_1)
- net 3.3v: now also U1.4 (FB), R7.1; no longer U5.3 (EN)
- net GND: now also H1.1, H2.1, H3.1, H4.1, J3.2 (Pin_2)
- net dac_BCK: now also U5.31 (IO19); no longer U5.7 (IO35)
- net dac_DIN: now also U5.30 (IO18); no longer U5.6 (IO34)
- net dac_LRCK: now also U5.28 (IO17); no longer U5.9 (IO33)
- net at TP6.1, U2.1 (V_{IN}), U3.1 (V_{IN})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: now also U4.4 (FB)
- net at J1.1 (Pin_1): now also U5.25 (IO0); no longer U5.26 (IO4)
- net at J1.10 (Pin_10): now also U5.23 (IO15); no longer U5.31 (IO19)
- net at J1.2 (Pin_2): now also U5.35 (TXD0/IO1); no longer U5.29 (IO5)
- net at J1.3 (Pin_3): now also U5.24 (IO2); no longer U5.14 (IO12)
- net at J1.4 (Pin_4): now also U5.34 (RXD0/IO3); no longer U5.16 (IO13)
- net at J1.5 (Pin_5): now also U5.26 (IO4); no longer U5.13 (IO14)
- net at J1.6 (Pin_6): now also U5.29 (IO5); no longer U5.23 (IO15)
- net at J1.7 (Pin_7): now also U5.14 (IO12); no longer U5.27 (IO16)
- net at J1.8 (Pin_8): now also U5.16 (IO13); no longer U5.28 (IO17)
- net at J1.9 (Pin_9): now also U5.13 (IO14); no longer U5.30 (IO18)
- new net: R7.2, U5.3 (EN)
Other:
- moved on the sheet: J1

Commit message: a
Changed lines of the file:
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@@
 		(in_pos_files yes)
 		(dnp no)
-		(fields_autoplaced yes)
 		(property "Reference" "C7"
-			(at 156.21 115.5699 0)
+			(at 151.13 115.316 0)
 			(show_name no)
 			(do_not_autoplace no)
@@
 		)
 		(property "Value" "C2.2"
-			(at 156.21 118.1099 0)
+			(at 150.368 117.856 0)
 			(show_name no)
 			(do_not_autoplace no)
@@
 		(in_pos_files yes)
 		(dnp no)
-		(fields_autoplaced yes)
 		(property "Reference" "C5"
-			(at 146.05 115.5699 0)
+			(at 140.97 115.57 0)
 			(show_name no)
 			(do_not_autoplace no)
@@
 		)
 		(property "Value" "C2.2"
-			(at 146.05 118.1099 0)
+			(at 140.208 118.11 0)
 			(show_name no)
 			(do_not_autoplace no)
@@
 		(in_pos_files yes)
 		(dnp no)
-		(fields_autoplaced yes)
 		(property "Reference" "C6"
-			(at 151.13 115.5699 0)
+			(at 146.05 115.316 0)
 			(show_name no)
 			(do_not_autoplace no)
@@
 		)
 		(property "Value" "C2.2"
-			(at 151.13 118.1099 0)
+			(at 145.542 118.11 0)
 			(show_name no)
 			(do_not_autoplace no)
@@
 		(in_pos_files yes)
 		(dnp no)
-		(fields_autoplaced yes)
 		(property "Reference" "C8"
-			(at 161.29 115.5699 0)
+			(at 156.21 115.316 0)
 			(show_name no)
 			(do_not_autoplace no)
@@
 		)
 		(property "Value" "C2.2"
-			(at 161.29 118.1099 0)
-			(show_name no)
-			(do_not_autoplace no)
+			(at 155.194 118.11 0)
+			(show_name no)
+			(do_not_autoplace no)
