File: inkBT.kicad_pcb (KiCad board)
At the start: 2 copper layers, 34 parts, among them J1 Conn_01x03, J2 Conn_01x10, J3 Conn_01x06, U1 LM2596S-5, U2 ESP32-WROOM-32, U3 PCM5102A, U5 LM2596S-3.3, U6 ME6211C33M5, U7 ME6211C33M5

Commit message: a
Parts:
- added H1: MountingHole_Pad, MountingHole:MountingHole_2.5mm_Pad_Via, F.Cu at (148.8, 41.0)
- added H2: MountingHole_Pad, MountingHole:MountingHole_2.5mm_Pad_Via, F.Cu at (149.9, 102.3)
- added H3: MountingHole_Pad, MountingHole:MountingHole_2.5mm_Pad_Via, F.Cu at (48.4, 93.9)
- added H4: MountingHole_Pad, MountingHole:MountingHole_2.5mm_Pad_Via, F.Cu at (45.7, 40.6)
- added R7: R100K, Resistor_SMD:R_1206_3216Metric_Pad1.30x1.75mm_HandSolder, F.Cu at (55.9, 40.6)
- J3: value Conn_01x06 -> Conn_01x02; footprint Connector_PinHeader_2.00mm:PinHeader_1x06_P2.00mm_Vertical -> Connector_PinHeader_2.54mm:PinHeader_1x02_P2.54mm_Vertical
- moved TP1 80.1 mm to (45.5, 70.3)
- moved TP2 80.1 mm to (45.5, 78.4)
- moved TP3 80.1 mm to (49.5, 66.3)
- moved TP4 80.1 mm to (45.5, 66.3)
- moved TP5 80.1 mm to (45.5, 74.4)
- moved TP6 80.1 mm to (49.5, 74.4)
- moved TP7 80.1 mm to (49.5, 70.3)
- moved C7 60.3 mm to (138.1, 68.6), turned to 180 degrees
- moved R2 58.2 mm to (137.2, 73.7)
- moved R5 57.7 mm to (137.2, 71.1)
- moved C8 57.2 mm to (138.1, 76.2), turned to 180 degrees
- moved R6 55.3 mm to (95.5, 64.5), turned to 180 degrees
- moved J3 50.4 mm to (104.1, 40.6)
- moved R4 48.7 mm to (95.5, 67.8), turned to 180 degrees
- moved C6 44.7 mm to (135.6, 86.4)
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- renumbered C8 to C1, C9 to C10, C12 to C11, C10 to C12, C7 to C2, C6 to C3, C5 to C4, C1 to C5, C2 to C6, C3 to C7, C4 to C8, C11 to C9, J2 to J1, J1 to J2, R6 to R1, R1 to R5, R5 to R6, TP2 to TP1, TP4 to TP2, TP5 to TP3, TP1 to TP4, TP3 to TP5, TP7 to TP6, TP6 to TP7, U5 to U1, U7 to U2, U6 to U3, U1 to U4, U2 to U5, U3 to U6
Connections:
- J1 pad 1: Net-(J2-Pin_1) -> Net-(J1-Pin_1)
- J1 pad 10: Net-(J2-Pin_10) -> Net-(J1-Pin_10)
- J1 pad 2: Net-(J2-Pin_2) (its old number) -> Net-(J1-Pin_2)
- J1 pad 3: Net-(J2-Pin_3) (its old number) -> Net-(J1-Pin_3)
- J1 pad 4: Net-(J2-Pin_4) -> Net-(J1-Pin_4)
- J1 pad 5: Net-(J2-Pin_5) -> Net-(J1-Pin_5)
- J1 pad 6: Net-(J2-Pin_6) -> Net-(J1-Pin_6)
- J1 pad 7: Net-(J2-Pin_7) -> Net-(J1-Pin_7)
- J1 pad 8: Net-(J2-Pin_8) -> Net-(J1-Pin_8)
- J1 pad 9: Net-(J2-Pin_9) -> Net-(J1-Pin_9)
- J3 pad 1: Net-(J3-Pin_1) -> +12V
- J3 pad 2: Net-(J3-Pin_2) -> GND
- TP6 pad 1: Net-(U1-OUT) -> Net-(U2-V_{IN})
- U1 pad 4: unconnected-(U5-FB-Pad4) -> 3.3v
- U2 pad 1: Net-(U1-OUT) -> Net-(U2-V_{IN})
- U3 pad 1: Net-(U1-OUT) -> Net-(U2-V_{IN})
- U4 pad 2: Net-(U1-OUT) -> Net-(U2-V_{IN})
- U4 pad 4: unconnected-(U1-FB-Pad4) -> Net-(U2-V_{IN})
- U5 pad 13: Net-(J2-Pin_5) -> Net-(J1-Pin_9)
- U5 pad 14: Net-(J2-Pin_3) (its old number) -> Net-(J1-Pin_7)
- U5 pad 16: Net-(J2-Pin_4) -> Net-(J1-Pin_8)
- U5 pad 17: Net-(J3-Pin_4) -> unconnected-(U5-SHD/SD2-Pad17)
- U5 pad 18: Net-(J3-Pin_3) -> unconnected-(U5-SWP/SD3-Pad18)
- U5 pad 19: Net-(J3-Pin_1) -> unconnected-(U5-SCS/CMD-Pad19)
- U5 pad 20: Net-(J3-Pin_2) -> unconnected-(U5-SCK/CLK-Pad20)
- U5 pad 21: Net-(J3-Pin_5) -> unconnected-(U5-SDO/SD0-Pad21)
- U5 pad 22: Net-(J3-Pin_6) -> unconnected-(U5-SDI/SD1-Pad22)
- U5 pad 23: Net-(J2-Pin_6) -> Net-(J1-Pin_10)
- U5 pad 24: unconnected-(U2-IO2-Pad24) -> Net-(J1-Pin_3)
- U5 pad 25: unconnected-(U2-IO0-Pad25) -> Net-(J1-Pin_1)
- U5 pad 26: Net-(J2-Pin_1) -> Net-(J1-Pin_5)
- U5 pad 27: Net-(J2-Pin_7) -> unconnected-(U5-IO16-Pad27)
- U5 pad 28: Net-(J2-Pin_8) -> dac_LRCK
- U5 pad 29: Net-(J2-Pin_2) (its old number) -> Net-(J1-Pin_6)
- U5 pad 3: 3.3v -> Net-(U5-EN)
- U5 pad 30: Net-(J2-Pin_9) -> dac_DIN
- U5 pad 31: Net-(J2-Pin_10) -> dac_BCK
- U5 pad 34: unconnected-(U2-RXD0/IO3-Pad34) -> Net-(J1-Pin_4)
- U5 pad 35: unconnected-(U2-TXD0/IO1-Pad35) -> Net-(J1-Pin_2)
- U5 pad 6: dac_DIN -> unconnected-(U5-IO34-Pad6)
- U5 pad 7: dac_BCK -> unconnected-(U5-IO35-Pad7)
- U5 pad 9: dac_LRCK -> unconnected-(U5-IO33-Pad9)
Routing:
- net Net-(J2-Pin_2): track 0.00 -> 14.4 mm
- net Net-(J2-Pin_3): track 0.00 -> 14.2 mm
- net Net-(U6-OUTR): track 0.00 -> 8.94 mm
- net Net-(U6-OUTL): track 0.00 -> 8.42 mm

Commit message: a
Parts:
- moved H2 129.8 mm to (28.6, 55.9)
- moved H4 107.8 mm to (134.6, 101.6)
- moved U3 77.7 mm to (49.4, 85.4), turned to 0 degrees
- moved U4 73.3 mm to (54.3, 71.4)
- moved U2 72.6 mm to (49.4, 80.3), turned to 0 degrees
- moved U1 68.8 mm to (54.3, 58.7)
- moved J3 67.3 mm to (38.1, 53.3)
- moved R1 64.7 mm to (68.6, 62.5), turned to -90 degrees
- moved TP2 37.1 mm to (17.8, 53.8)
- moved TP5 37.1 mm to (17.8, 49.8)
- moved TP6 37.1 mm to (21.8, 49.8)
- moved TP1 37.1 mm to (17.8, 45.7)
- moved TP3 37.1 mm to (21.8, 41.7)
- moved TP4 37.1 mm to (17.8, 41.7)
- moved TP7 37.1 mm to (21.8, 45.7)
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Connections:
- J3 pad 1: +12V -> GND
- J3 pad 2: GND -> +12V
Routing:
- net 3.3v: track 0.00 -> 43.1 mm
- net +12V: track 0.00 -> 26.2 mm
- net Net-(U2-V_{IN}): track 0.00 -> 25.6 mm
- net Net-(J2-Pin_2): track 14.4 -> 0.00 mm
- net Net-(J2-Pin_3): track 14.2 -> 0.00 mm
- net Net-(U6-OUTR): track 8.94 -> 0.00 mm
- net Net-(U6-OUTL): track 8.42 -> 0.00 mm
Other:
- board outline added: 5.1 x 3.1 mm

Commit message: a
Parts:
- added ?: LOGO, LOGO, F.Cu at (120.0, 69.8)
- added ?: LOGO, LOGO, F.Cu at (58.4, 100.3)
- added ?: LOGO, LOGO, B.Cu at (45.3, 80.6)
- added ?: LOGO, LOGO, B.Cu at (95.9, 100.3)
- moved TP3 53.9 mm to (58.4, 81.3)
- moved TP4 52.9 mm to (64.8, 66.0)
- moved TP2 46.2 mm to (54.0, 82.5)
- moved TP7 45.6 mm to (41.3, 87.0)
- moved TP6 35.6 mm to (40.6, 80.0)
- moved TP1 23.4 mm to (37.5, 58.4)
- moved TP5 19.1 mm to (31.8, 62.9)
- moved H3 5.27 mm to (31.1, 98.4)
- moved U2 5.09 mm to (49.7, 85.4)
- moved U3 5.08 mm to (49.4, 80.3)
- moved H4 3.17 mm to (134.6, 98.4)
- moved H2 2.51 mm to (31.1, 55.9)
- moved H1 0.92 mm to (134.6, 55.2)
- turned R3 to -90 degrees
- turned R4 to -90 degrees
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Routing:
- net 3.3v Ddac: track 0.00 -> 86.2 mm
- net 3.3v Adac: track 0.00 -> 80.5 mm
- net EN_dac: track 0.00 -> 79.3 mm
- net Net-(J1-Pin_7): track 0.00 -> 51.8 mm, vias 0 -> 4
- net Net-(J1-Pin_9): track 0.00 -> 51.1 mm, vias 0 -> 4
- net Net-(J1-Pin_8): track 0.00 -> 43.5 mm, vias 0 -> 4
- net Net-(J1-Pin_3): track 0.00 -> 36.5 mm, vias 0 -> 4
- net Net-(J1-Pin_1): track 0.00 -> 35.0 mm, vias 0 -> 2
- net Net-(J1-Pin_5): track 0.00 -> 28.9 mm, vias 0 -> 2
- net dac_BCK: track 0.00 -> 28.4 mm
- net Net-(J1-Pin_10): track 0.00 -> 27.7 mm, vias 0 -> 2
- net dac_DIN: track 0.00 -> 25.4 mm
- net Net-(J1-Pin_4): track 0.00 -> 24.5 mm
- net Net-(J1-Pin_6): track 0.00 -> 24.3 mm, vias 0 -> 2
- net Net-(J1-Pin_2): track 0.00 -> 23.7 mm
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- added copper zone on B.Cu, net GND
- added copper zone on F.Cu, net GND
Other:
- board size 5.1 x 3.1 mm -> 112 x 51 mm
